Commit message: trying to get gazebo talking to ros control

File: ros/src/clam/clam_description/urdf/clam.xacro (robot description, xacro)
@@ -16,4 +16,5 @@
   <property name="M_PI" value="3.14159"/>
   <!-- TABLETOP LINK -->
+  <!--
   <joint name="tabletop_joint" type="fixed">
     <origin xyz="0 0 0" rpy="0 0 0" />
@@ -44,11 +45,17 @@
     <material>Gazebo/White</material>
   </gazebo>
+  -->
+  <link name="world" />
+  <joint name="fixed" type="fixed">
+    <parent link="world" />
+    <child link="base_link" />
+  </joint>
   <!-- BASE LINK -->
   <link name="base_link">
-    <!--inertial>
-        <origin xyz="0 0 0" />
-        <mass value="1.0" />
-        <inertia  ixx="1.0" ixy="0.0"  ixz="0.0"  iyy="100.0"  iyz="0.0"  izz="1.0" />
-        </inertial-->
+    <inertial>
+      <origin xyz="0 0 0" />
+      <mass value="1.0" />
+      <inertia  ixx="1.0" ixy="0.0"  ixz="0.0"  iyy="100.0"  iyz="0.0"  izz="1.0" />
+    </inertial>
     <visual>
       <origin xyz="0 0 0" rpy="${M_PI/2} 0 0" /> <!-- rotate PI/2 -->

Commit message: adding basic scaffolding to slim model and splitting out clam to more easily allow import into other URDFs

File: ros/src/clam/clam_description/urdf/clam.xacro (robot description, xacro)
@@ -15,66 +15,29 @@
   <property name="M_SCALE" value="0.001 0.001 0.001"/>
   <property name="M_PI" value="3.14159"/>
-  <!-- TABLETOP LINK -->
-  <!--
-  <joint name="tabletop_joint" type="fixed">
-    <origin xyz="0 0 0" rpy="0 0 0" />
-    <parent link="base_link"/>
-    <child link="tabletop_link"/>
-  </joint>
-  <link name="tabletop_link">
-    <inertial>
-      <origin xyz=" 0 0 -0.017"/>
-      <mass value="100.0" />
-      <inertia  ixx="1.0" ixy="0.0"  ixz="0.0"  iyy="100.0"  iyz="0.0"  izz="1.0" />
-    </inertial>
-    <visual>
-      <origin xyz=" 0 0 -0.017"  rpy="${.5*M_PI} 0 ${.5*M_PI}"/>
-      <geometry>
-        <mesh filename="package://clam_description/stl/tabletop_link.STL" scale="${M_SCALE}" />
-      </geometry>
-      <material name="Brown" />
-    </visual>
-    <collision>
-      <origin xyz=" 0 0 -0.017"  rpy="${.5*M_PI} 0 ${.5*M_PI}"/>
-      <geometry>
-        <mesh filename="package://clam_description/stl/tabletop_link_simple.STL" scale="${M_SCALE}" />
+  <link name="arm_base_link">
+    <inertial>
+      <origin xyz="0 0 0" />
+      <mass value="1.0" />
+      <inertia  ixx="1.0" ixy="0.0"  ixz="0.0"  iyy="100.0"  iyz="0.0"  izz="1.0" />
+    </inertial>
+    <visual>
+      <origin xyz="0 0 0" rpy="${M_PI/2} 0 0" /> <!-- rotate PI/2 -->
+      <geometry>
+        <mesh filename="package://clam_description/stl/base_link.STL" scale="${M_SCALE}" />
+      </geometry>
+      <material name="Grey" />
+    </visual>
+    <collision>
+      <origin xyz="0 0 0" rpy="${M_PI/2} 0 0" /> <!-- rotate PI/2 -->
+      <geometry>
+        <mesh filename="package://clam_description/stl/base_link_simple.STL" scale="${M_SCALE}" />
       </geometry>
       </collision>>
   </link>
-  <gazebo reference="tabletop_link">
-    <material>Gazebo/White</material>
-  </gazebo>
-  -->
-  <link name="world" />
-  <joint name="fixed" type="fixed">
-    <parent link="world" />
-    <child link="base_link" />
-  </joint>
-  <!-- BASE LINK -->
-  <link name="base_link">
-    <inertial>
-      <origin xyz="0 0 0" />
-      <mass value="1.0" />
-      <inertia  ixx="1.0" ixy="0.0"  ixz="0.0"  iyy="100.0"  iyz="0.0"  izz="1.0" />
-    </inertial>
-    <visual>
-      <origin xyz="0 0 0" rpy="${M_PI/2} 0 0" /> <!-- rotate PI/2 -->
-      <geometry>
-        <mesh filename="package://clam_description/stl/base_link.STL" scale="${M_SCALE}" />
-      </geometry>
-      <material name="Grey" />
-    </visual>
-    <collision>
-      <origin xyz="0 0 0" rpy="${M_PI/2} 0 0" /> <!-- rotate PI/2 -->
-      <geometry>
-        <mesh filename="package://clam_description/stl/base_link_simple.STL" scale="${M_SCALE}" />
-      </geometry>
-      </collision>>
-  </link>
-  <gazebo reference="base_link">
+  <gazebo reference="arm_base_link">
     <material>Gazebo/Grey</material>
   </gazebo>
   <joint name="shoulder_pan_joint" type="revolute">
-    <parent link="base_link"/>
+    <parent link="arm_base_link"/>
     <child link="shoulder_pan_link"/>
     <origin xyz="0 0 0.05" rpy="0 ${M_PI/2} ${M_PI*0}" />
@@ -548,5 +511,6 @@
   </gazebo>
   <!-- FAKE CAMERA CALIBRATION POINT AT GRIPPER TIP -->
-  <!--joint name="gripper_fake_tip_joint" type="fixed">
+  <!--
+  <joint name="gripper_fake_tip_joint" type="fixed">
     <origin xyz="0.1785 0.0 0.0" rpy="0 0 0" />
     <parent link="gripper_roll_link"/>
@@ -574,4 +538,5 @@
   <gazebo reference="gripper_fake_tip_link">
     <material>Gazebo/Grey</material>
-  </gazebo-->
+  </gazebo>
+  -->
 </robot>

File: ros/src/clam/clam_description/urdf/materials.urdf.xacro (robot description, xacro)
@@ -13,4 +13,7 @@
         <color rgba="0.2 0.2 0.2 1.0"/>
     </material>
+    <material name="LightGrey">
+        <color rgba="0.6 0.6 0.6 1.0"/>
+    </material>
     <material name="Orange">
         <color rgba="${255/255} ${108/255} ${10/255} 1.0"/>

File: ros/src/slim_description/urdf/slim.urdf.xacro (robot description, xacro)
@@ -1,5 +1,135 @@
 <?xml version="1.0"?>
 <robot xmlns:xacro="http://www.ros.org/wiki/xacro" name="slim">
+  <link name="base_link" />
+  <joint name="fixed" type="fixed">
+    <parent link="base_link" />
+    <child link="lift_base" />
+  </joint>
+  <link name="lift_base">
+    <visual>
+      <geometry>
+        <box size="1.3 0.2 0.01" />
+      </geometry>
+      <material name="LightGrey" />
+    </visual>
+  </link>
+  <gazebo reference="lift_base">
+    <material>Gazebo/LightGrey</material>
+  </gazebo>
+  <joint name="lift_base_joint" type="fixed">
+    <parent link="lift_base" />
+    <child link="fl_lift_rod" />
+  </joint>
+  <link name="fl_lift_rod">
+    <visual>
+      <origin xyz="0.55 0.07 0.3" rpy="0 0 0" />
+      <geometry>
+        <cylinder length="0.6" radius="0.01" />
+      </geometry>
+      <material name="LightGrey" />
+    </visual>
+  </link>
+  <joint name="fl_lift_joint" type="prismatic">
+    <axis xyz="0 0 1" />
+    <parent link="fl_lift_rod" />
+    <child link="slide_rail_base" />
+    <limit effort="1000.0" velocity="0.1" lower="0" upper="0.5" />
+  </joint>
+  <link name="fr_lift_rod">
+    <visual>
+      <origin xyz="-0.55 0.07 0.3" rpy="0 0 0" />
+      <geometry>
+        <cylinder length="0.6" radius="0.01" />
+      </geometry>
+      <material name="LightGrey" />
+    </visual>
+  </link>
+  <joint name="fr_lift_joint" type="fixed">
+    <parent link="lift_base" />
+    <child link="fr_lift_rod" />
+  </joint>
+  <link name="bl_lift_rod">
+    <visual>
+      <origin xyz="0.55 -0.07 0.3" rpy="0 0 0" />
+      <geometry>
+        <cylinder length="0.6" radius="0.01" />
+      </geometry>
+      <material name="LightGrey" />
+    </visual>
+  </link>
+  <joint name="bl_lift_joint" type="fixed">
+    <parent link="lift_base" />
+    <child link="bl_lift_rod" />
+  </joint>
+  <link name="br_lift_rod">
+    <visual>
+      <origin xyz="-0.55 -0.07 0.3" rpy="0 0 0" />
+      <geometry>
+        <cylinder length="0.6" radius="0.01" />
+      </geometry>
+      <material name="LightGrey" />
+    </visual>
+  </link>
+  <joint name="br_lift_joint" type="fixed">
+    <parent link="lift_base" />
+    <child link="br_lift_rod" />
+  </joint>
+  <link name="l_lift_rod_cap">
+    <visual>
+      <origin xyz="0.55 0 0.6" />
+      <geometry>
+        <box size="0.05 0.2 0.01" />
+      </geometry>
+      <material name="LightGrey" />
+    </visual>
+  </link>
+  <joint name="l_lift_rod_cap_joint" type="fixed">
+    <parent link="fl_lift_rod" />
+    <child link="l_lift_rod_cap" />
+  </joint>
+  <link name="r_lift_rod_cap">
+    <visual>
+      <origin xyz="-0.55 0 0.6" />
+      <geometry>
+        <box size="0.05 0.2 0.01" />
+      </geometry>
+      <material name="LightGrey" />
+    </visual>
+  </link>
+  <joint name="r_lift_rod_cap_joint" type="fixed">
+    <parent link="fr_lift_rod" />
+    <child link="r_lift_rod_cap" />
+  </joint>
+  <link name="slide_rail_base">
+    <visual>
+      <origin xyz="0 0 0.01" />
+      <geometry>
+        <box size="1.2 0.2 0.01" />
+      </geometry>
+      <material name="LightGrey" />
+    </visual>
+  </link>
+  <gazebo reference="slide_rail_base">
+    <material>Gazebo/LightGrey</material>
+  </gazebo>
+  <joint name="slide_rail_base_joint" type="prismatic">
+    <axis xyz="1 0 0" />
+    <parent link="slide_rail_base" />
+    <child link="slide_rail" />
+    <limit effort="1000.0" velocity="0.2" lower="-0.4" upper="0.4" />
+  </joint>
+  <link name="slide_rail">
+    <visual>
+      <geometry>
+        <box size="0.18 0.18 0.01" />
+      </geometry>
+      <material name="LightGrey" />
+      <origin xyz="0 0 0.02" />
+    </visual>
+  </link>
+  <joint name="slide_rail_joint" type="fixed">
+    <parent link="slide_rail" />
+    <child link="arm_base_link" />
+  </joint>
   <xacro:include filename="$(find clam_description)/urdf/clam.xacro" />
-  <xacro:clam name="clamarm" />
 </robot>

Commit message: working on pick and place demo

File: ros/src/clam/clam_description/urdf/clam.xacro (robot description, xacro)
@@ -424,80 +424,80 @@
   </gazebo>
   <!-- Transmissions for ROS Control -->
-  <transmission name="tran1">
+  <transmission name="shoulder_pan_trans">
     <type>transmission_interface/SimpleTransmission</type>
     <joint name="shoulder_pan_joint">
       <hardwareInterface>EffortJointInterface</hardwareInterface>
     </joint>
-    <actuator name="motor1">
-      <hardwareInterface>EffortJointInterface</hardwareInterface>
-      <mechanicalReduction>1</mechanicalReduction>
-    </actuator>
-  </transmission>
-  <transmission name="tran1">
+    <actuator name="shoulder_pan_motor">
+      <hardwareInterface>EffortJointInterface</hardwareInterface>
+      <mechanicalReduction>1</mechanicalReduction>
+    </actuator>
+  </transmission>
+  <transmission name="shoulder_pitch_trans">
     <type>transmission_interface/SimpleTransmission</type>
     <joint name="shoulder_pitch_joint">
       <hardwareInterface>EffortJointInterface</hardwareInterface>
     </joint>
-    <actuator name="motor1">
-      <hardwareInterface>EffortJointInterface</hardwareInterface>
-      <mechanicalReduction>1</mechanicalReduction>
-    </actuator>
-  </transmission>
-  <transmission name="tran1">
+    <actuator name="shoulder_pitch_motor">
+      <hardwareInterface>EffortJointInterface</hardwareInterface>
+      <mechanicalReduction>1</mechanicalReduction>
+    </actuator>
+  </transmission>
+  <transmission name="elbow_roll_trans">
     <type>transmission_interface/SimpleTransmission</type>
     <joint name="elbow_roll_joint">
       <hardwareInterface>EffortJointInterface</hardwareInterface>
     </joint>
-    <actuator name="motor1">
-      <hardwareInterface>EffortJointInterface</hardwareInterface>
-      <mechanicalReduction>1</mechanicalReduction>
-    </actuator>
-  </transmission>
-  <transmission name="tran1">
+    <actuator name="elbow_roll_motor">
+      <hardwareInterface>EffortJointInterface</hardwareInterface>
+      <mechanicalReduction>1</mechanicalReduction>
+    </actuator>
+  </transmission>
+  <transmission name="elbow_pitch_trans">
     <type>transmission_interface/SimpleTransmission</type>
     <joint name="elbow_pitch_joint">
       <hardwareInterface>EffortJointInterface</hardwareInterface>
     </joint>
-    <actuator name="motor1">
-      <hardwareInterface>EffortJointInterface</hardwareInterface>
-      <mechanicalReduction>1</mechanicalReduction>
-    </actuator>
-  </transmission>
-  <transmission name="tran1">
+    <actuator name="elbow_pitch_motor">
+      <hardwareInterface>EffortJointInterface</hardwareInterface>
+      <mechanicalReduction>1</mechanicalReduction>
+    </actuator>
+  </transmission>
+  <transmission name="wrist_roll_trans">
     <type>transmission_interface/SimpleTransmission</type>
     <joint name="wrist_roll_joint">
       <hardwareInterface>EffortJointInterface</hardwareInterface>
     </joint>
-    <actuator name="motor1">
-      <hardwareInterface>EffortJointInterface</hardwareInterface>
-      <mechanicalReduction>1</mechanicalReduction>
-    </actuator>
-  </transmission>
-  <transmission name="tran1">
+    <actuator name="wrist_roll_motor">
+      <hardwareInterface>EffortJointInterface</hardwareInterface>
+      <mechanicalReduction>1</mechanicalReduction>
+    </actuator>
+  </transmission>
+  <transmission name="wrist_pitch_trans">
     <type>transmission_interface/SimpleTransmission</type>
     <joint name="wrist_pitch_joint">
       <hardwareInterface>EffortJointInterface</hardwareInterface>
     </joint>
-    <actuator name="motor1">
-      <hardwareInterface>EffortJointInterface</hardwareInterface>
-      <mechanicalReduction>1</mechanicalReduction>
-    </actuator>
-  </transmission>
-  <transmission name="tran1">
+    <actuator name="wrist_pitch_motor">
+      <hardwareInterface>EffortJointInterface</hardwareInterface>
+      <mechanicalReduction>1</mechanicalReduction>
+    </actuator>
+  </transmission>
+  <transmission name="gripper_roll_trans">
     <type>transmission_interface/SimpleTransmission</type>
     <joint name="gripper_roll_joint">
       <hardwareInterface>EffortJointInterface</hardwareInterface>
     </joint>
-    <actuator name="motor1">
-      <hardwareInterface>EffortJointInterface</hardwareInterface>
-      <mechanicalReduction>1</mechanicalReduction>
-    </actuator>
-  </transmission>
-  <transmission name="tran1">
+    <actuator name="gripper_roll_motor">
+      <hardwareInterface>EffortJointInterface</hardwareInterface>
+      <mechanicalReduction>1</mechanicalReduction>
+    </actuator>
+  </transmission>
+  <transmission name="gripper_finger_trans">
     <type>transmission_interface/SimpleTransmission</type>
     <joint name="gripper_finger_joint">
       <hardwareInterface>EffortJointInterface</hardwareInterface>
     </joint>
-    <actuator name="motor1">
+    <actuator name="gripper_finger_motor">
       <hardwareInterface>EffortJointInterface</hardwareInterface>
       <mechanicalReduction>1</mechanicalReduction>

File: ros/src/slim_description/urdf/slim.urdf.xacro (robot description, xacro)
@@ -13,4 +13,13 @@
       <material name="LightGrey" />
     </visual>
+    <collision>
+      <geometry>
+        <box size="1.3 0.2 0.01" />
+      </geometry>
+    </collision>
+    <inertial>
+      <mass value="5" />
+      <inertia />
+    </inertial>
   </link>
   <gazebo reference="lift_base">

Commit message: working moveit+rviz+gazebo!

File: ros/src/clam/clam_description/urdf/clam.xacro (robot description, xacro)
@@ -504,4 +504,54 @@
     </actuator>
   </transmission>
+  <transmission name="r_gripper_aft_trans">
+    <type>transmission_interface/SimpleTransmission</type>
+    <joint name="r_gripper_aft_joint">
+      <hardwareInterface>PositionJointInterface</hardwareInterface>
+    </joint>
+    <actuator name="r_gripper_aft_motor">
+      <hardwareInterface>PositionJointInterface</hardwareInterface>
+      <mechanicalReduction>1</mechanicalReduction>
+    </actuator>
+  </transmission>
+  <transmission name="l_gripper_fwd_trans">
+    <type>transmission_interface/SimpleTransmission</type>
+    <joint name="l_gripper_fwd_joint">
+      <hardwareInterface>PositionJointInterface</hardwareInterface>
+    </joint>
+    <actuator name="l_gripper_fwd_motor">
+      <hardwareInterface>PositionJointInterface</hardwareInterface>
+      <mechanicalReduction>1</mechanicalReduction>
+    </actuator>
+  </transmission>
+  <transmission name="r_gripper_fwd_trans">
+    <type>transmission_interface/SimpleTransmission</type>
+    <joint name="r_gripper_fwd_joint">
+      <hardwareInterface>PositionJointInterface</hardwareInterface>
+    </joint>
+    <actuator name="r_gripper_fwd_motor">
+      <hardwareInterface>PositionJointInterface</hardwareInterface>
+      <mechanicalReduction>1</mechanicalReduction>
+    </actuator>
+  </transmission>
+  <transmission name="gripper_finger_pincher_trans">
+    <type>transmission_interface/SimpleTransmission</type>
+    <joint name="gripper_finger_pincher_joint">
+      <hardwareInterface>PositionJointInterface</hardwareInterface>
+    </joint>
+    <actuator name="gripper_finger_pincher_motor">
+      <hardwareInterface>PositionJointInterface</hardwareInterface>
+      <mechanicalReduction>1</mechanicalReduction>
+    </actuator>
+  </transmission>
+  <transmission name="r_gripper_aft_pincher_trans">
+    <type>transmission_interface/SimpleTransmission</type>
+    <joint name="r_gripper_aft_pincher_joint">
+      <hardwareInterface>PositionJointInterface</hardwareInterface>
+    </joint>
+    <actuator name="r_gripper_aft_pincher_motor">
+      <hardwareInterface>PositionJointInterface</hardwareInterface>
+      <mechanicalReduction>1</mechanicalReduction>
+    </actuator>
+  </transmission>
   <!-- FAKE CAMERA CALIBRATION POINT AT GRIPPER TIP -->
   <!--
