Commit message: almost grasping

File: ros/src/clam/clam_description/urdf/clam.xacro (robot description, xacro)
@@ -288,12 +288,12 @@
     <material>Gazebo/Grey</material>
   </gazebo>
-  <joint name="r_gripper_aft_joint" type="revolute">
+  <joint name="r_gripper_aft_joint" type="fixed">
     <parent link="gripper_roll_link"/>
     <child link="r_gripper_aft_link"/>
     <origin xyz="0.026 -0.011  0" rpy="${1.345*M_PI} ${M_PI/2} ${34.58*M_PI/180}" />
-    <axis xyz="1 0 0" />
-    <limit effort="300" velocity="1" lower="-3.14" upper="3.14" />
-    <mimic joint="gripper_finger_joint" multiplier="-1.0" offset="0.0" />
-    <dynamics damping="50" friction="1"/>
+    <!-- <axis xyz="1 0 0" /> -->
+    <!-- <limit effort="300" velocity="1" lower="-3.14" upper="3.14" /> -->
+    <!-- <mimic joint="gripper_finger_joint" multiplier="-1.0" offset="0.0" /> -->
+    <!-- <dynamics damping="50" friction="1"/> -->
   </joint>
   <!-- RIGHT GRIPPER AFT LINK -->
@@ -315,66 +315,12 @@
     <material>Gazebo/Grey</material>
   </gazebo>
-  <joint name="l_gripper_fwd_joint" type="revolute">
-    <parent link="gripper_roll_link"/>
-    <child link="l_gripper_fwd_link"/>
-    <origin xyz="0.05 0.008 0.007" rpy="${M_PI*(1+.04)} ${M_PI/2} ${214.58*M_PI/180}" />
-    <axis xyz="1 0 0" />
-    <limit effort="300" velocity="1" lower="0" upper="1.57" />
-    <mimic joint="gripper_finger_joint" multiplier="1.0" offset="0.0" />
-    <dynamics damping="50" friction="1"/>
-  </joint>
-  <!-- LEFT GRIPPER FWD LINK -->
-  <link name="l_gripper_fwd_link">
-    <inertial>
-      <origin xyz="0 0 0"  />
-      <mass value="1.0" />
-      <inertia  ixx="1.0" ixy="0.0"  ixz="0.0"  iyy="100.0"  iyz="0.0"  izz="1.0" />
-    </inertial>
-    <visual>
-      <origin xyz="0 0 0" rpy="0 0 ${M_PI}" />
-      <geometry>
-        <mesh filename="package://clam_description/stl/l_gripper_fwd_link.STL" scale="1 1 1" />
-      </geometry>
-      <material name="Grey" />
-    </visual>
-  </link>
-  <gazebo reference="l_gripper_fwd_link">
-    <material>Gazebo/Grey</material>
-  </gazebo>
-  <joint name="r_gripper_fwd_joint" type="revolute">
-    <parent link="gripper_roll_link"/>
-    <child link="r_gripper_fwd_link"/>
-    <origin xyz="0.05 -0.0014 0.007" rpy="${M_PI*(1-.04)} ${M_PI/2} ${145.42*M_PI/180}" />
-    <axis xyz="1 0 0" />
-    <limit effort="300" velocity="1" lower="-1.57" upper="0" />
-    <mimic joint="gripper_finger_joint" multiplier="-1.0" offset="0.0" />
-    <dynamics damping="50" friction="1"/>
-  </joint>
-  <!-- RIGHT GRIPPER FWD LINK -->
-  <link name="r_gripper_fwd_link">
-    <inertial>
-      <origin xyz="0 0 0"  />
-      <mass value="1.0" />
-      <inertia  ixx="1.0" ixy="0.0"  ixz="0.0"  iyy="100.0"  iyz="0.0"  izz="1.0" />
-    </inertial>
-    <visual>
-      <origin xyz="0 0 0" rpy="0 0 ${M_PI}" />
-      <geometry>
-        <mesh filename="package://clam_description/stl/r_gripper_fwd_link.STL" scale="1 1 1" />
-      </geometry>
-      <material name="Grey" />
-    </visual>
-  </link>
-  <gazebo reference="r_gripper_fwd_link">
-    <material>Gazebo/Grey</material>
-  </gazebo>
-  <joint name="gripper_finger_pincher_joint" type="revolute">
+  <joint name="gripper_finger_pincher_joint" type="fixed">
     <parent link="gripper_finger_link"/>
     <child link="l_gripper_pincher_link"/>
     <origin xyz="-0.0032 0 -0.0508" rpy="${203.27*M_PI/180-.3150*M_PI} 0 0" />
-    <axis xyz="1 0 0" />
-    <limit effort="300" velocity="1" lower="-1.57" upper="1.57" />
-    <mimic joint="gripper_finger_joint" multiplier="-1.0" offset="0.0" />
-    <dynamics damping="50" friction="1"/>
+    <!-- <axis xyz="1 0 0" /> -->
+    <!-- <limit effort="300" velocity="1" lower="-1.57" upper="1.57" /> -->
+    <!-- <mimic joint="gripper_finger_joint" multiplier="-1.0" offset="0.0" /> -->
+    <!-- <dynamics damping="50" friction="1"/> -->
   </joint>
   <!-- LEFT GRIPPER PINCHER -->
@@ -396,12 +342,12 @@
     <material>Gazebo/Black</material>
   </gazebo>
-  <joint name="r_gripper_aft_pincher_joint" type="revolute">
+  <joint name="r_gripper_aft_pincher_joint" type="fixed">
     <parent link="r_gripper_aft_link"/>
     <child link="r_gripper_pincher_link"/>
     <origin xyz="0 0 -0.0508" rpy="${23.27*M_PI/180-.3150*M_PI} ${M_PI} 0" />
-    <axis xyz="1 0 0" />
-    <limit effort="300" velocity="1" lower="0" upper="1.57" />
-    <mimic joint="gripper_finger_joint" multiplier="-1.0" offset="0.0" />
-    <dynamics damping="50" friction="1"/>
+    <!-- <axis xyz="1 0 0" /> -->
+    <!-- <limit effort="300" velocity="1" lower="0" upper="1.57" /> -->
+    <!-- <mimic joint="gripper_finger_joint" multiplier="-1.0" offset="0.0" /> -->
+    <!-- <dynamics damping="50" friction="1"/> -->
   </joint>
   <!-- RIGHT GRIPPER PINCHER -->
@@ -500,54 +446,4 @@
     </joint>
     <actuator name="gripper_finger_motor">
-      <hardwareInterface>PositionJointInterface</hardwareInterface>
-      <mechanicalReduction>1</mechanicalReduction>
-    </actuator>
-  </transmission>
-  <transmission name="r_gripper_aft_trans">
-    <type>transmission_interface/SimpleTransmission</type>
-    <joint name="r_gripper_aft_joint">
-      <hardwareInterface>PositionJointInterface</hardwareInterface>
-    </joint>
-    <actuator name="r_gripper_aft_motor">
-      <hardwareInterface>PositionJointInterface</hardwareInterface>
-      <mechanicalReduction>1</mechanicalReduction>
-    </actuator>
-  </transmission>
-  <transmission name="l_gripper_fwd_trans">
-    <type>transmission_interface/SimpleTransmission</type>
-    <joint name="l_gripper_fwd_joint">
-      <hardwareInterface>PositionJointInterface</hardwareInterface>
-    </joint>
-    <actuator name="l_gripper_fwd_motor">
-      <hardwareInterface>PositionJointInterface</hardwareInterface>
-      <mechanicalReduction>1</mechanicalReduction>
-    </actuator>
-  </transmission>
-  <transmission name="r_gripper_fwd_trans">
-    <type>transmission_interface/SimpleTransmission</type>
-    <joint name="r_gripper_fwd_joint">
-      <hardwareInterface>PositionJointInterface</hardwareInterface>
-    </joint>
-    <actuator name="r_gripper_fwd_motor">
-      <hardwareInterface>PositionJointInterface</hardwareInterface>
-      <mechanicalReduction>1</mechanicalReduction>
-    </actuator>
-  </transmission>
-  <transmission name="gripper_finger_pincher_trans">
-    <type>transmission_interface/SimpleTransmission</type>
-    <joint name="gripper_finger_pincher_joint">
-      <hardwareInterface>PositionJointInterface</hardwareInterface>
-    </joint>
-    <actuator name="gripper_finger_pincher_motor">
-      <hardwareInterface>PositionJointInterface</hardwareInterface>
-      <mechanicalReduction>1</mechanicalReduction>
-    </actuator>
-  </transmission>
-  <transmission name="r_gripper_aft_pincher_trans">
-    <type>transmission_interface/SimpleTransmission</type>
-    <joint name="r_gripper_aft_pincher_joint">
-      <hardwareInterface>PositionJointInterface</hardwareInterface>
-    </joint>
-    <actuator name="r_gripper_aft_pincher_motor">
       <hardwareInterface>PositionJointInterface</hardwareInterface>
       <mechanicalReduction>1</mechanicalReduction>

File: ros/src/slim_description/urdf/slim.urdf (robot description, URDF)
Before this commit: robot slim, 30 links, 29 joints
Links:
- removed link l_gripper_fwd_link
- removed link r_gripper_fwd_link
Joints:
- removed joint l_gripper_fwd_joint
- removed joint r_gripper_fwd_joint
- joint gripper_finger_pincher_joint: axis 1 0 0 -> (none); limit lower=-1.57 upper=1.57 effort=300 velocity=1 -> (none); mimic joint=gripper_finger_joint multiplier=-1.0 offset=0.0 -> (none); type revolute -> fixed
- joint r_gripper_aft_joint: axis 1 0 0 -> (none); limit lower=-3.14 upper=3.14 effort=300 velocity=1 -> (none); mimic joint=gripper_finger_joint multiplier=-1.0 offset=0.0 -> (none); type revolute -> fixed
- joint r_gripper_aft_pincher_joint: axis 1 0 0 -> (none); limit lower=0 upper=1.57 effort=300 velocity=1 -> (none); mimic joint=gripper_finger_joint multiplier=-1.0 offset=0.0 -> (none); type revolute -> fixed
