Commit message: adding slim_moveit_config package with initial settings from MoveIt Setup Assistant

File: ros/src/slim_description/urdf/slim.urdf (robot description, URDF)
Before this commit: robot slim, 17 links, 16 joints
Links:
- removed link world
- added link arm_base_link, mass 1.0; collision mesh filename=package://clam_description/stl/base_link_simple.STL scale=0.001 0.001 0.001; visual mesh filename=package://clam_description/stl/base_link.STL scale=0.001 0.001 0.001
- added link bl_lift_rod; visual cylinder length=0.6 radius=0.01
- added link br_lift_rod; visual cylinder length=0.6 radius=0.01
- added link fl_lift_rod; visual cylinder length=0.6 radius=0.01
- added link fr_lift_rod; visual cylinder length=0.6 radius=0.01
- added link l_lift_rod_cap; visual box size=0.05 0.2 0.01
- added link lift_base; visual box size=1.3 0.2 0.01
- added link r_lift_rod_cap; visual box size=0.05 0.2 0.01
- link base_link: mass 1.0 -> None; geometry 
- link slide_rail_base: geometry visual box size=1.2 0.2 0.01
Joints:
- added joint bl_lift_joint: type fixed, parent lift_base, child bl_lift_rod
- added joint br_lift_joint: type fixed, parent lift_base, child br_lift_rod
- added joint fl_lift_joint: type prismatic, parent fl_lift_rod, child slide_rail_base, axis 0 0 1, limit lower=0 upper=0.5 effort=1000.0 velocity=0.1
- added joint fr_lift_joint: type fixed, parent lift_base, child fr_lift_rod
- added joint l_lift_rod_cap_joint: type fixed, parent fl_lift_rod, child l_lift_rod_cap
- added joint lift_base_joint: type fixed, parent lift_base, child fl_lift_rod
- added joint r_lift_rod_cap_joint: type fixed, parent fr_lift_rod, child r_lift_rod_cap
- joint fixed: child slide_rail_base -> lift_base; parent world -> base_link
- joint shoulder_pan_joint: parent base_link -> arm_base_link
- joint slide_rail_base_joint: limit lower=-0.41 upper=0.41 effort=1000.0 velocity=0.2 -> lower=-0.4 upper=0.4 effort=1000.0 velocity=0.2
- joint slide_rail_joint: child base_link -> arm_base_link

Commit message: and physical properties to new URDF links and re-running setup assistant

File: ros/src/slim_description/urdf/slim.urdf (robot description, URDF)
Before this commit: robot slim, 24 links, 23 joints
Links:
- added link back_frame, mass 5; collision box size=1.12 0.02 0.02; visual box size=1.12 0.02 0.02
- added link bl_frame_post, mass 5; collision box size=0.02 0.02 0.6; visual box size=0.02 0.02 0.6
- added link br_frame_post, mass 5; collision box size=0.02 0.02 0.6; visual box size=0.02 0.02 0.6
- added link fl_frame_post, mass 5; collision box size=0.02 0.02 0.6; visual box size=0.02 0.02 0.6
- added link fr_frame_post, mass 5; collision box size=0.02 0.02 0.6; visual box size=0.02 0.02 0.6
- link bl_lift_rod: mass None -> 5; geometry collision cylinder length=0.6 radius=0.01; visual cylinder length=0.6 radius=0.01
- link br_lift_rod: mass None -> 5; geometry collision cylinder length=0.6 radius=0.01; visual cylinder length=0.6 radius=0.01
- link fl_lift_rod: mass None -> 5; geometry collision cylinder length=0.6 radius=0.01; visual cylinder length=0.6 radius=0.01
- link fr_lift_rod: mass None -> 5; geometry collision cylinder length=0.6 radius=0.01; visual cylinder length=0.6 radius=0.01
- link l_lift_rod_cap: mass None -> 5; geometry collision box size=0.05 0.2 0.01; visual box size=0.05 0.8 0.01
- link lift_base: mass None -> 5; geometry collision box size=1.3 0.8 0.01; visual box size=1.3 0.8 0.01
- link r_lift_rod_cap: mass None -> 5; geometry collision box size=0.05 0.2 0.01; visual box size=0.05 0.8 0.01
- link slide_rail: mass None -> 5; geometry collision box size=0.18 0.18 0.01; visual box size=0.18 0.18 0.01
- link slide_rail_base: mass None -> 5; geometry collision box size=1.2 0.2 0.01; visual box size=1.2 0.2 0.01
Joints:
- added joint back_frame_joint: type fixed, parent l_lift_rod_cap, child back_frame
- added joint bl_frame_post_joint: type fixed, parent lift_base, child bl_frame_post
- added joint br_frame_post_joint: type fixed, parent lift_base, child br_frame_post
- added joint fl_frame_post_joint: type fixed, parent lift_base, child fl_frame_post
- added joint fr_frame_post_joint: type fixed, parent lift_base, child fr_frame_post

File: ros/src/slim_description/urdf/slim.urdf.xacro (robot description, xacro)
@@ -41,4 +41,15 @@
       <material name="Grey" />
     </visual>
+    <collision>
+      <origin xyz="0.55 0.14 0.3" />
+      <geometry>
+        <box size="0.02 0.02 0.6" />
+      </geometry>
+    </collision>
+    <inertial>
+      <origin xyz="0.55 0.14 0.3" />
+      <mass value="5" />
+      <inertia ixx="1.0" ixy="0.0" ixz="0.0" iyy="100.0" iyz="0.0" izz="1.0"/>
+    </inertial>
   </link>
   <gazebo reference="fl_frame_post">
@@ -57,4 +68,15 @@
       <material name="Grey" />
     </visual>
+    <collision>
+      <origin xyz="-0.55 0.14 0.3" />
+      <geometry>
+        <box size="0.02 0.02 0.6" />
+      </geometry>
+    </collision>
+    <inertial>
+      <origin xyz="-0.55 0.14 0.3" />
+      <mass value="5" />
+      <inertia ixx="1.0" ixy="0.0" ixz="0.0" iyy="100.0" iyz="0.0" izz="1.0"/>
+    </inertial>
   </link>
   <gazebo reference="fr_frame_post">
@@ -73,4 +95,15 @@
       <material name="Grey" />
     </visual>
+    <collision>
+      <origin xyz="0.55 -0.64 0.3" />
+      <geometry>
+        <box size="0.02 0.02 0.6" />
+      </geometry>
+    </collision>
+    <inertial>
+      <origin xyz="0.55 -0.64 0.3" />
+      <mass value="5" />
+      <inertia ixx="1.0" ixy="0.0" ixz="0.0" iyy="100.0" iyz="0.0" izz="1.0"/>
+    </inertial>
   </link>
   <gazebo reference="bl_frame_post">
@@ -89,4 +122,15 @@
       <material name="Grey" />
     </visual>
+    <collision>
+      <origin xyz="-0.55 -0.64 0.3" />
+      <geometry>
+        <box size="0.02 0.02 0.6" />
+      </geometry>
+    </collision>
+    <inertial>
+      <origin xyz="-0.55 -0.64 0.3" />
+      <mass value="5" />
+      <inertia ixx="1.0" ixy="0.0" ixz="0.0" iyy="100.0" iyz="0.0" izz="1.0"/>
+    </inertial>
   </link>
   <gazebo reference="br_frame_post">
@@ -211,4 +255,15 @@
       <material name="Grey" />
     </visual>
+    <collision>
+      <origin xyz="0 -0.64 0.595" />
+      <geometry>
+        <box size="1.12 0.02 0.02" />
+      </geometry>
+    </collision>
+    <inertial>
+      <origin xyz="0 -0.64 0.595" />
+      <mass value="5" />
+      <inertia ixx="1.0" ixy="0.0" ixz="0.0" iyy="100.0" iyz="0.0" izz="1.0"/>
+    </inertial>
   </link>
   <gazebo reference="back_frame">

Commit message: MoveIt setup changes

File: ros/src/slim_description/urdf/slim.urdf (robot description, URDF)
Before this commit: robot slim, 29 links, 28 joints
Links:
- added link camera, mass 0.1; collision box size=0.05 0.05 0.05; visual box size=0.05 0.05 0.05
Joints:
- added joint camera_joint: type fixed, parent back_frame, child camera

Commit message: fixing camera

File: ros/src/slim_description/urdf/slim.urdf (robot description, URDF)
Before this commit: robot slim, 28 links, 27 joints
Joints:
- joint camera_joint: axis (none) -> 0 1 0; origin (none) -> xyz=0 -0.64 0.595 rpy=0 0 1.57
