Commit message: Importing stock clam arm into slim urdf

File: ros/src/slim_description/urdf/slim.urdf.xacro (robot description, xacro)
@@ -1,26 +1,5 @@
 <?xml version="1.0"?>
 <robot xmlns:xacro="http://www.ros.org/wiki/xacro" name="slim">
-  <property name="box_width" value="0.75" />
-  <link name="box">
-    <inertial>
-      <origin xyz="0 0 0" />
-      <mass value="1.0" />
-      <inertia ixx="1.0" ixy="0.0" ixz="0.0" iyy="100.0" iyz="0.0" izz="1.0" />
-    </inertial>
-    <visual>
-      <origin xyz="0 0 0"/>
-      <geometry>
-        <box size="${box_width} ${box_width} ${box_width}" />
-      </geometry>
-    </visual>
-    <collision>
-      <origin xyz="0 0 0"/>
-      <geometry>
-        <box size="${box_width} ${box_width} ${box_width}" />
-      </geometry>
-    </collision>
-  </link>
-  <gazebo reference="box">
-    <material>Gazebo/Blue</material>
-  </gazebo>
+  <xacro:include filename="$(find clam_description)/urdf/clam.xacro" />
+  <xacro:clam name="clamarm" />
 </robot>

Commit message: commenting out broken xml in urdf

File: ros/src/slim_description/urdf/slim.urdf.xacro (robot description, xacro)
@@ -18,8 +18,8 @@
       </geometry>
     </collision>
-    <inertial>
-      <mass value="5" />
-      <inertia />
-    </inertial>
+    <!-- <inertial> -->
+    <!--   <mass value="5" /> -->
+    <!--   <inertia /> -->
+    <!-- </inertial> -->
   </link>
   <gazebo reference="lift_base">

Commit message: dummy inertia values

File: ros/src/slim_description/urdf/slim.urdf.xacro (robot description, xacro)
@@ -18,8 +18,8 @@
       </geometry>
     </collision>
-    <!-- <inertial> -->
-    <!--   <mass value="5" /> -->
-    <!--   <inertia /> -->
-    <!-- </inertial> -->
+    <inertial>
+      <mass value="5" />
+      <inertia ixx="1.0" ixy="0.0" ixz="0.0" iyy="100.0" iyz="0.0" izz="1.0"/>
+    </inertial>
   </link>
   <gazebo reference="lift_base">
@@ -38,4 +38,14 @@
       <material name="LightGrey" />
     </visual>
+    <collision>
+      <origin xyz="0.55 0.07 0.3" rpy="0 0 0" />
+      <geometry>
+        <cylinder length="0.6" radius="0.01" />
+      </geometry>
+    </collision>
+    <inertial>
+      <mass value="5" />
+      <inertia ixx="1.0" ixy="0.0" ixz="0.0" iyy="100.0" iyz="0.0" izz="1.0"/>
+    </inertial>
   </link>
   <joint name="fl_lift_joint" type="prismatic">
@@ -53,4 +63,14 @@
       <material name="LightGrey" />
     </visual>
+    <collision>
+      <origin xyz="-0.55 0.07 0.3" rpy="0 0 0" />
+      <geometry>
+        <cylinder length="0.6" radius="0.01" />
+      </geometry>
+    </collision>
+    <inertial>
+      <mass value="5" />
+      <inertia ixx="1.0" ixy="0.0" ixz="0.0" iyy="100.0" iyz="0.0" izz="1.0"/>
+    </inertial>
   </link>
   <joint name="fr_lift_joint" type="fixed">
@@ -66,4 +86,14 @@
       <material name="LightGrey" />
     </visual>
+    <collision>
+      <origin xyz="0.55 -0.07 0.3" rpy="0 0 0" />
+      <geometry>
+        <cylinder length="0.6" radius="0.01" />
+      </geometry>
+    </collision>
+    <inertial>
+      <mass value="5" />
+      <inertia ixx="1.0" ixy="0.0" ixz="0.0" iyy="100.0" iyz="0.0" izz="1.0"/>
+    </inertial>
   </link>
   <joint name="bl_lift_joint" type="fixed">
@@ -79,4 +109,14 @@
       <material name="LightGrey" />
     </visual>
+    <collision>
+      <origin xyz="-0.55 -0.07 0.3" rpy="0 0 0" />
+      <geometry>
+        <cylinder length="0.6" radius="0.01" />
+      </geometry>
+    </collision>
+    <inertial>
+      <mass value="5" />
+      <inertia ixx="1.0" ixy="0.0" ixz="0.0" iyy="100.0" iyz="0.0" izz="1.0"/>
+    </inertial>
   </link>
   <joint name="br_lift_joint" type="fixed">
@@ -92,4 +132,14 @@
       <material name="LightGrey" />
     </visual>
+    <collision>
+      <origin xyz="0.55 0 0.6" />
+      <geometry>
+        <box size="0.05 0.2 0.01" />
+      </geometry>
+    </collision>
+    <inertial>
+      <mass value="5" />
+      <inertia ixx="1.0" ixy="0.0" ixz="0.0" iyy="100.0" iyz="0.0" izz="1.0"/>
+    </inertial>
   </link>
   <joint name="l_lift_rod_cap_joint" type="fixed">
@@ -105,4 +155,14 @@
       <material name="LightGrey" />
     </visual>
+    <collision>
+      <origin xyz="-0.55 0 0.6" />
+      <geometry>
+        <box size="0.05 0.2 0.01" />
+      </geometry>
+    </collision>
+    <inertial>
+      <mass value="5" />
+      <inertia ixx="1.0" ixy="0.0" ixz="0.0" iyy="100.0" iyz="0.0" izz="1.0"/>
+    </inertial>
   </link>
   <joint name="r_lift_rod_cap_joint" type="fixed">
@@ -118,4 +178,14 @@
       <material name="LightGrey" />
     </visual>
+    <collision>
+      <origin xyz="0 0 0.01" />
+      <geometry>
+        <box size="1.2 0.2 0.01" />
+      </geometry>
+    </collision>
+    <inertial>
+      <mass value="5" />
+      <inertia ixx="1.0" ixy="0.0" ixz="0.0" iyy="100.0" iyz="0.0" izz="1.0"/>
+    </inertial>
   </link>
   <gazebo reference="slide_rail_base">
@@ -136,4 +206,14 @@
       <origin xyz="0 0 0.02" />
     </visual>
+    <collision>
+      <geometry>
+        <box size="0.18 0.18 0.01" />
+      </geometry>
+      <origin xyz="0 0 0.02" />
+    </collision>
+    <inertial>
+      <mass value="5" />
+      <inertia ixx="1.0" ixy="0.0" ixz="0.0" iyy="100.0" iyz="0.0" izz="1.0"/>
+    </inertial>
   </link>
   <joint name="slide_rail_joint" type="fixed">

Commit message: adding transmissions for the gantry joints

File: ros/src/slim_description/urdf/slim.urdf.xacro (robot description, xacro)
@@ -221,4 +221,24 @@
     <child link="arm_base_link" />
   </joint>
+  <transmission name="fl_lift_trans">
+    <type>transmission_interface/SimpleTransmission</type>
+    <joint name="fl_lift_joint">
+      <hardwareInterface>EffortJointInterface</hardwareInterface>
+    </joint>
+    <actuator name="fl_lift_motor">
+      <hardwareInterface>EffortJointInterface</hardwareInterface>
+      <mechanicalReduction>1</mechanicalReduction>
+    </actuator>
+  </transmission>
+  <transmission name="slide_rail_base_trans">
+    <type>transmission_interface/SimpleTransmission</type>
+    <joint name="slide_rail_base_joint">
+      <hardwareInterface>EffortJointInterface</hardwareInterface>
+    </joint>
+    <actuator name="slide_rail_base_motor">
+      <hardwareInterface>EffortJointInterface</hardwareInterface>
+      <mechanicalReduction>1</mechanicalReduction>
+    </actuator>
+  </transmission>
   <xacro:include filename="$(find clam_description)/urdf/clam.xacro" />
 </robot>

Commit message: more little fixes for pick and place

File: ros/src/slim_description/urdf/slim.urdf.xacro (robot description, xacro)
@@ -23,7 +23,4 @@
     </inertial>
   </link>
-  <gazebo reference="lift_base">
-    <material>Gazebo/LightGrey</material>
-  </gazebo>
   <joint name="lift_base_joint" type="fixed">
     <parent link="lift_base" />
@@ -189,7 +186,4 @@
     </inertial>
   </link>
-  <gazebo reference="slide_rail_base">
-    <material>Gazebo/LightGrey</material>
-  </gazebo>
   <joint name="slide_rail_base_joint" type="prismatic">
     <axis xyz="1 0 0" />

Commit message: modifications to URDF to make it look more realistic

File: ros/src/slim_description/urdf/slim.urdf.xacro (robot description, xacro)
@@ -8,19 +8,89 @@
   <link name="lift_base">
     <visual>
-      <geometry>
-        <box size="1.3 0.2 0.01" />
-      </geometry>
-      <material name="LightGrey" />
-    </visual>
-    <collision>
-      <geometry>
-        <box size="1.3 0.2 0.01" />
-      </geometry>
-    </collision>
-    <inertial>
-      <mass value="5" />
-      <inertia ixx="1.0" ixy="0.0" ixz="0.0" iyy="100.0" iyz="0.0" izz="1.0"/>
-    </inertial>
-  </link>
+      <origin xyz="0 -0.25 0" />
+      <geometry>
+        <box size="1.3 0.8 0.01" />
+      </geometry>
+      <material name="Grey" />
+    </visual>
+    <collision>
+      <origin xyz="0 -0.35 0" />
+      <geometry>
+        <box size="1.3 0.8 0.01" />
+      </geometry>
+    </collision>
+    <inertial>
+      <origin xyz="0 -0.35 0" />
+      <mass value="5" />
+      <inertia ixx="1.0" ixy="0.0" ixz="0.0" iyy="100.0" iyz="0.0" izz="1.0"/>
+    </inertial>
+  </link>
+  <gazebo reference="lift_base">
+    <material>Gazebo/Grey</material>
+  </gazebo>
+  <joint name="fl_frame_post_joint" type="fixed">
+    <parent link="lift_base" />
+    <child link="fl_frame_post" />
+  </joint>
+  <link name="fl_frame_post">
+    <visual>
+      <origin xyz="0.55 0.14 0.3" />
+      <geometry>
+        <box size="0.02 0.02 0.6" />
+      </geometry>
+      <material name="Grey" />
+    </visual>
+  </link>
+  <gazebo reference="fl_frame_post">
+    <material>Gazebo/Grey</material>
+  </gazebo>
+  <joint name="fr_frame_post_joint" type="fixed">
+    <parent link="lift_base" />
+    <child link="fr_frame_post" />
+  </joint>
+  <link name="fr_frame_post">
+    <visual>
+      <origin xyz="-0.55 0.14 0.3" />
+      <geometry>
+        <box size="0.02 0.02 0.6" />
+      </geometry>
+      <material name="Grey" />
+    </visual>
+  </link>
+  <gazebo reference="fr_frame_post">
+    <material>Gazebo/Grey</material>
+  </gazebo>
+  <joint name="bl_frame_post_joint" type="fixed">
+    <parent link="lift_base" />
+    <child link="bl_frame_post" />
+  </joint>
+  <link name="bl_frame_post">
+    <visual>
+      <origin xyz="0.55 -0.64 0.3" />
+      <geometry>
+        <box size="0.02 0.02 0.6" />
+      </geometry>
+      <material name="Grey" />
+    </visual>
+  </link>
+  <gazebo reference="bl_frame_post">
+    <material>Gazebo/Grey</material>
+  </gazebo>
+  <joint name="br_frame_post_joint" type="fixed">
+    <parent link="lift_base" />
+    <child link="br_frame_post" />
+  </joint>
+  <link name="br_frame_post">
+    <visual>
+      <origin xyz="-0.55 -0.64 0.3" />
+      <geometry>
+        <box size="0.02 0.02 0.6" />
+      </geometry>
+      <material name="Grey" />
+    </visual>
+  </link>
+  <gazebo reference="br_frame_post">
+    <material>Gazebo/Grey</material>
+  </gazebo>
   <joint name="lift_base_joint" type="fixed">
     <parent link="lift_base" />
@@ -33,5 +103,5 @@
         <cylinder length="0.6" radius="0.01" />
       </geometry>
-      <material name="LightGrey" />
+      <material name="Grey" />
     </visual>
     <collision>
@@ -46,4 +116,7 @@
     </inertial>
   </link>
+  <gazebo reference="fl_lift_rod">
+    <material>Gazebo/Grey</material>
+  </gazebo>
   <joint name="fl_lift_joint" type="prismatic">
     <axis xyz="0 0 1" />
@@ -58,5 +131,5 @@
         <cylinder length="0.6" radius="0.01" />
       </geometry>
-      <material name="LightGrey" />
+      <material name="Grey" />
     </visual>
     <collision>
@@ -71,4 +144,7 @@
     </inertial>
   </link>
+  <gazebo reference="fr_lift_rod">
+    <material>Gazebo/Grey</material>
+  </gazebo>
   <joint name="fr_lift_joint" type="fixed">
     <parent link="lift_base" />
@@ -81,5 +157,5 @@
         <cylinder length="0.6" radius="0.01" />
       </geometry>
-      <material name="LightGrey" />
+      <material name="Grey" />
     </visual>
     <collision>
@@ -94,4 +170,7 @@
     </inertial>
   </link>
+  <gazebo reference="bl_lift_rod">
+    <material>Gazebo/Grey</material>
+  </gazebo>
   <joint name="bl_lift_joint" type="fixed">
     <parent link="lift_base" />
@@ -104,5 +183,5 @@
         <cylinder length="0.6" radius="0.01" />
       </geometry>
-      <material name="LightGrey" />
+      <material name="Grey" />
     </visual>
     <collision>
@@ -117,27 +196,49 @@
     </inertial>
   </link>
+  <gazebo reference="br_lift_rod">
+    <material>Gazebo/Grey</material>
+  </gazebo>
   <joint name="br_lift_joint" type="fixed">
     <parent link="lift_base" />
     <child link="br_lift_rod" />
   </joint>
+  <link name="back_frame">
+    <visual>
+      <origin xyz="0 -0.64 0.595" />
+      <geometry>
+        <box size="1.12 0.02 0.02" />
+      </geometry>
+      <material name="Grey" />
+    </visual>
+  </link>
+  <gazebo reference="back_frame">
+    <material>Gazebo/Grey</material>
+  </gazebo>
+  <joint name="back_frame_joint" type="fixed">
+    <parent link="l_lift_rod_cap" />
+    <child link="back_frame" />
+  </joint>
   <link name="l_lift_rod_cap">
     <visual>
+      <origin xyz="0.55 -0.25 0.6" />
+      <geometry>
+        <box size="0.05 0.8 0.01" />
+      </geometry>
+      <material name="Grey" />
+    </visual>
+    <collision>
       <origin xyz="0.55 0 0.6" />
       <geometry>
         <box size="0.05 0.2 0.01" />
       </geometry>
-      <material name="LightGrey" />
-    </visual>
-    <collision>
-      <origin xyz="0.55 0 0.6" />
-      <geometry>
-        <box size="0.05 0.2 0.01" />
-      </geometry>
-    </collision>
-    <inertial>
-      <mass value="5" />
-      <inertia ixx="1.0" ixy="0.0" ixz="0.0" iyy="100.0" iyz="0.0" izz="1.0"/>
-    </inertial>
-  </link>
+    </collision>
+    <inertial>
+      <mass value="5" />
+      <inertia ixx="1.0" ixy="0.0" ixz="0.0" iyy="100.0" iyz="0.0" izz="1.0"/>
+    </inertial>
+  </link>
+  <gazebo reference="l_lift_rod_cap">
+    <material>Gazebo/Grey</material>
+  </gazebo>
   <joint name="l_lift_rod_cap_joint" type="fixed">
     <parent link="fl_lift_rod" />
@@ -146,21 +247,24 @@
   <link name="r_lift_rod_cap">
     <visual>
+      <origin xyz="-0.55 -0.25 0.6" />
+      <geometry>
+        <box size="0.05 0.8 0.01" />
+      </geometry>
+      <material name="Grey" />
+    </visual>
+    <collision>
       <origin xyz="-0.55 0 0.6" />
       <geometry>
         <box size="0.05 0.2 0.01" />
       </geometry>
-      <material name="LightGrey" />
-    </visual>
-    <collision>
-      <origin xyz="-0.55 0 0.6" />
-      <geometry>
-        <box size="0.05 0.2 0.01" />
-      </geometry>
-    </collision>
-    <inertial>
-      <mass value="5" />
-      <inertia ixx="1.0" ixy="0.0" ixz="0.0" iyy="100.0" iyz="0.0" izz="1.0"/>
-    </inertial>
-  </link>
+    </collision>
+    <inertial>
+      <mass value="5" />
+      <inertia ixx="1.0" ixy="0.0" ixz="0.0" iyy="100.0" iyz="0.0" izz="1.0"/>
+    </inertial>
+  </link>
+  <gazebo reference="r_lift_rod_cap">
+    <material>Gazebo/Grey</material>
+  </gazebo>
   <joint name="r_lift_rod_cap_joint" type="fixed">
     <parent link="fr_lift_rod" />
@@ -173,5 +277,5 @@
         <box size="1.2 0.2 0.01" />
       </geometry>
-      <material name="LightGrey" />
+      <material name="Grey" />
     </visual>
     <collision>
@@ -186,4 +290,7 @@
     </inertial>
   </link>
+  <gazebo reference="slide_rail_base">
+    <material>Gazebo/Grey</material>
+  </gazebo>
   <joint name="slide_rail_base_joint" type="prismatic">
     <axis xyz="1 0 0" />
@@ -197,5 +304,5 @@
         <box size="0.18 0.18 0.01" />
       </geometry>
-      <material name="LightGrey" />
+      <material name="Grey" />
       <origin xyz="0 0 0.02" />
     </visual>
@@ -211,4 +318,7 @@
     </inertial>
   </link>
+  <gazebo reference="slide_rail">
+    <material>Gazebo/Grey</material>
+  </gazebo>
   <joint name="slide_rail_joint" type="fixed">
     <parent link="slide_rail" />

Commit message: using slightly more sane inertia values - still need to update mass

File: ros/src/slim_description/urdf/slim.urdf.xacro (robot description, xacro)
@@ -1,4 +1,5 @@
 <?xml version="1.0"?>
 <robot xmlns:xacro="http://www.ros.org/wiki/xacro" name="slim">
+  <xacro:include filename="$(find slim_description)/urdf/macros.xacro" />
   <link name="base_link" />
   <joint name="fixed" type="fixed">
@@ -23,5 +24,5 @@
       <origin xyz="0 -0.35 0" />
       <mass value="5" />
-      <inertia ixx="1.0" ixy="0.0" ixz="0.0" iyy="100.0" iyz="0.0" izz="1.0"/>
+      <box_inertia m="5" x="1.3" y="0.8" z="0.01" />
     </inertial>
   </link>
@@ -50,5 +51,5 @@
       <origin xyz="0.55 0.14 0.3" />
       <mass value="5" />
-      <inertia ixx="1.0" ixy="0.0" ixz="0.0" iyy="100.0" iyz="0.0" izz="1.0"/>
+      <box_inertia m="5" x="0.02" y="0.02" z="0.6" />
     </inertial>
   </link>
@@ -77,5 +78,5 @@
       <origin xyz="-0.55 0.14 0.3" />
       <mass value="5" />
-      <inertia ixx="1.0" ixy="0.0" ixz="0.0" iyy="100.0" iyz="0.0" izz="1.0"/>
+      <box_inertia m="5" x="0.02" y="0.02" z="0.6" />
     </inertial>
   </link>
@@ -104,5 +105,5 @@
       <origin xyz="0.55 -0.64 0.3" />
       <mass value="5" />
-      <inertia ixx="1.0" ixy="0.0" ixz="0.0" iyy="100.0" iyz="0.0" izz="1.0"/>
+      <box_inertia m="5" x="0.02" y="0.02" z="0.6" />
     </inertial>
   </link>
@@ -131,5 +132,5 @@
       <origin xyz="-0.55 -0.64 0.3" />
       <mass value="5" />
-      <inertia ixx="1.0" ixy="0.0" ixz="0.0" iyy="100.0" iyz="0.0" izz="1.0"/>
+      <box_inertia m="5" x="0.02" y="0.02" z="0.6" />
     </inertial>
   </link>
@@ -157,5 +158,5 @@
     <inertial>
       <mass value="5" />
-      <inertia ixx="1.0" ixy="0.0" ixz="0.0" iyy="100.0" iyz="0.0" izz="1.0"/>
+      <cylinder_inertia m="5" r="0.01" h="0.6" />
     </inertial>
   </link>
@@ -185,5 +186,5 @@
     <inertial>
       <mass value="5" />
-      <inertia ixx="1.0" ixy="0.0" ixz="0.0" iyy="100.0" iyz="0.0" izz="1.0"/>
+      <cylinder_inertia m="5" r="0.01" h="0.6" />
     </inertial>
   </link>
@@ -211,5 +212,5 @@
     <inertial>
       <mass value="5" />
-      <inertia ixx="1.0" ixy="0.0" ixz="0.0" iyy="100.0" iyz="0.0" izz="1.0"/>
+      <cylinder_inertia m="5" r="0.01" h="0.6" />
     </inertial>
   </link>
@@ -237,5 +238,5 @@
     <inertial>
       <mass value="5" />
-      <inertia ixx="1.0" ixy="0.0" ixz="0.0" iyy="100.0" iyz="0.0" izz="1.0"/>
+      <cylinder_inertia m="5" r="0.01" h="0.6" />
     </inertial>
   </link>
@@ -264,5 +265,5 @@
       <origin xyz="0 -0.64 0.595" />
       <mass value="5" />
-      <inertia ixx="1.0" ixy="0.0" ixz="0.0" iyy="100.0" iyz="0.0" izz="1.0"/>
+      <box_inertia m="5" x="1.12" y="0.02" z="0.02" />
     </inertial>
   </link>
@@ -290,5 +291,5 @@
     <inertial>
       <mass value="5" />
-      <inertia ixx="1.0" ixy="0.0" ixz="0.0" iyy="100.0" iyz="0.0" izz="1.0"/>
+      <box_inertia m="5" x="0.05" y="0.2" z="0.01" />
     </inertial>
   </link>
@@ -316,5 +317,5 @@
     <inertial>
       <mass value="5" />
-      <inertia ixx="1.0" ixy="0.0" ixz="0.0" iyy="100.0" iyz="0.0" izz="1.0"/>
+      <box_inertia m="5" x="0.05" y="0.8" z="0.01" />
     </inertial>
   </link>
@@ -342,5 +343,5 @@
     <inertial>
       <mass value="5" />
-      <inertia ixx="1.0" ixy="0.0" ixz="0.0" iyy="100.0" iyz="0.0" izz="1.0"/>
+      <box_inertia m="5" x="1.2" y="0.2" z="0.01" />
     </inertial>
   </link>
@@ -370,5 +371,5 @@
     <inertial>
       <mass value="5" />
-      <inertia ixx="1.0" ixy="0.0" ixz="0.0" iyy="100.0" iyz="0.0" izz="1.0"/>
+      <box_inertia m="5" x="0.18" y="0.18" z="0.01" />
     </inertial>
   </link>

Commit message: adding a camera to the back of the frame

File: ros/src/slim_description/urdf/slim.urdf.xacro (robot description, xacro)
@@ -2,4 +2,7 @@
 <robot xmlns:xacro="http://www.ros.org/wiki/xacro" name="slim">
   <xacro:include filename="$(find slim_description)/urdf/macros.xacro" />
+  <xacro:property name="PI" value="3.1415926535897931"/>
+  <xacro:property name="cameraSize" value="0.05"/>
+  <xacro:property name="cameraMass" value="0.1"/>
   <link name="base_link" />
   <joint name="fixed" type="fixed">
@@ -274,4 +277,28 @@
     <parent link="l_lift_rod_cap" />
     <child link="back_frame" />
+  </joint>
+  <link name="camera">
+    <collision>
+      <origin xyz="0 -0.64 0.595" rpy="0 0 0"/>
+      <geometry>
+        <box size="${cameraSize} ${cameraSize} ${cameraSize}"/>
+      </geometry>
+    </collision>
+    <visual>
+      <origin xyz="0 -0.64 0.595" rpy="0 0 0"/>
+      <geometry>
+        <box size="${cameraSize} ${cameraSize} ${cameraSize}"/>
+      </geometry>
+      <material name="blue"/>
+    </visual>
+    <inertial>
+      <mass value="${cameraMass}" />
+      <origin xyz="0 -0.64 0.595" rpy="0 0 0"/>
+      <box_inertia m="${cameraMass}" x="${cameraSize}" y="${cameraSize}" z="${cameraSize}" />
+    </inertial>
+  </link>
+  <joint name="camera_joint" type="fixed">
+    <parent link="back_frame" />
+    <child link="camera" />
   </joint>
   <link name="l_lift_rod_cap">
@@ -408,3 +435,36 @@
     </plugin>
   </gazebo>
+  <!-- http://www.generationrobots.com/en/content/75-gazebo-and-ros -->
+  <gazebo reference="camera">
+    <material>Gazebo/Blue</material>
+    <sensor type="camera" name="camera1">
+      <update_rate>30.0</update_rate>
+      <camera name="head">
+        <horizontal_fov>1.3962634</horizontal_fov>
+        <image>
+          <width>800</width>
+          <height>800</height>
+          <format>R8G8B8</format>
+        </image>
+        <clip>
+          <near>0.02</near>
+          <far>300</far>
+        </clip>
+      </camera>
+      <plugin name="camera_controller" filename="libgazebo_ros_camera.so">
+        <alwaysOn>true</alwaysOn>
+        <updateRate>0.0</updateRate>
+        <cameraName>slim/camera1</cameraName>
+        <imageTopicName>image_raw</imageTopicName>
+        <cameraInfoTopicName>camera_info</cameraInfoTopicName>
+        <frameName>camera_link</frameName>
+        <hackBaseline>0.07</hackBaseline>
+        <distortionK1>0.0</distortionK1>
+        <distortionK2>0.0</distortionK2>
+        <distortionK3>0.0</distortionK3>
+        <distortionT1>0.0</distortionT1>
+        <distortionT2>0.0</distortionT2>
+      </plugin>
+    </sensor>
+  </gazebo>
 </robot>
