Commit message: working on pick place

File: ros/src/slim_description/urdf/slim.urdf.xacro (robot description, xacro)
@@ -280,5 +280,6 @@
   <link name="camera">
     <collision>
-      <origin xyz="0 -0.64 0.595" rpy="0 0 0"/>
+      <!-- <origin xyz="0 -0.64 0.595" rpy="0 0 0"/> -->
+      <origin xyz="0 0 0" rpy="0 0 0" />
       <geometry>
         <box size="${cameraSize} ${cameraSize} ${cameraSize}"/>
@@ -286,5 +287,6 @@
     </collision>
     <visual>
-      <origin xyz="0 -0.64 0.595" rpy="0 0 0"/>
+      <!-- <origin xyz="0 -0.64 0.595" rpy="0 0 0"/> -->
+      <origin xyz="0 0 0" rpy="0 0 0" />
       <geometry>
         <box size="${cameraSize} ${cameraSize} ${cameraSize}"/>
@@ -294,5 +296,6 @@
     <inertial>
       <mass value="${cameraMass}" />
-      <origin xyz="0 -0.64 0.595" rpy="0 0 0"/>
+      <!-- <origin xyz="0 -0.64 0.595" rpy="0 0 0"/> -->
+      <origin xyz="0 0 0" rpy="0 0 0" />
       <box_inertia m="${cameraMass}" x="${cameraSize}" y="${cameraSize}" z="${cameraSize}" />
     </inertial>
@@ -301,4 +304,7 @@
     <parent link="back_frame" />
     <child link="camera" />
+    <axis xyz="0 1 0" />
+    <origin xyz="0 -0.64 0.595" rpy="0 0 1.57"/>
+    <!-- <origin xyz="0 -0.64 0.595" rpy="-1.57 0 1.57"/> -->
   </joint>
   <link name="l_lift_rod_cap">
@@ -434,4 +440,20 @@
       <robotNamespace>/slim</robotNamespace>
     </plugin>
+  </gazebo>
+  <!-- http://answers.gazebosim.org/question/4324/gripper-tag-gazebophysicsgripper-doesnt-create-the/ -->
+  <gazebo>
+    <gripper name="grasping">
+        <grasp_check>
+            <attach_steps>20</attach_steps>
+            <detach_steps>40</detach_steps>
+            <min_contact_count>1</min_contact_count>
+        </grasp_check>
+        <!-- seem to only be able to specify one of these gripper_links -->
+        <!-- <gripper_link>gripper_finger_link</gripper_link> -->
+        <gripper_link>l_gripper_pincher_link</gripper_link>
+        <!-- <gripper_link>r_gripper_aft_link</gripper_link> -->
+        <!-- <gripper_link>r_gripper_pincher_link</gripper_link> -->
+        <palm_link>r_gripper_pincher_link</palm_link>
+    </gripper>
   </gazebo>
   <!-- http://www.generationrobots.com/en/content/75-gazebo-and-ros -->

Commit message: last minute changes

File: ros/src/slim_description/urdf/slim.urdf.xacro (robot description, xacro)
@@ -283,5 +283,5 @@
       <origin xyz="0 0 0" rpy="0 0 0" />
       <geometry>
-        <box size="${cameraSize} ${cameraSize} ${cameraSize}"/>
+        <box size="0.05 0.2 0.05" />
       </geometry>
     </collision>
@@ -290,5 +290,5 @@
       <origin xyz="0 0 0" rpy="0 0 0" />
       <geometry>
-        <box size="${cameraSize} ${cameraSize} ${cameraSize}"/>
+        <box size="0.05 0.2 0.05" />
       </geometry>
       <material name="blue"/>
@@ -305,5 +305,5 @@
     <child link="camera" />
     <axis xyz="0 1 0" />
-    <origin xyz="0 -0.64 0.595" rpy="0 0 1.57"/>
+    <origin xyz="0 -0.64 0.62" rpy="0 0 1.57"/>
     <!-- <origin xyz="0 -0.64 0.595" rpy="-1.57 0 1.57"/> -->
   </joint>

Commit message: changes from offfice

File: ros/src/slim_description/urdf/slim.urdf.xacro (robot description, xacro)
@@ -434,5 +434,5 @@
     </actuator>
   </transmission>
-  <xacro:include filename="$(find clam_description)/urdf/clam.xacro" />
+  <xacro:include filename="$(find slim_description)/urdf/slim_no_base.xacro" />
   <!-- ros_control plugin -->
   <gazebo>

File: ros/src/slim_description/urdf/slim_no_base.urdf (robot description, URDF)
Before this commit: robot slim, 28 links, 27 joints
Links:
- removed link back_frame
- removed link base_link
- removed link bl_frame_post
- removed link bl_lift_rod
- removed link br_frame_post
- removed link br_lift_rod
- removed link camera
- removed link fl_frame_post
- removed link fl_lift_rod
- removed link fr_frame_post
- removed link fr_lift_rod
- removed link l_lift_rod_cap
- removed link lift_base
- removed link r_lift_rod_cap
- removed link slide_rail
- removed link slide_rail_base
Joints:
- removed joint back_frame_joint
- removed joint bl_frame_post_joint
- removed joint bl_lift_joint
- removed joint br_frame_post_joint
- removed joint br_lift_joint
- removed joint camera_joint
- removed joint fixed
- removed joint fl_frame_post_joint
- removed joint fl_lift_joint
- removed joint fr_frame_post_joint
- removed joint fr_lift_joint
- removed joint l_lift_rod_cap_joint
- removed joint lift_base_joint
- removed joint r_lift_rod_cap_joint
- removed joint slide_rail_base_joint
- removed joint slide_rail_joint
- joint wrist_pitch_joint: limit lower=-1.9277025234 upper=1.7947575218 effort=300 velocity=1 -> lower=-0.0255663465 upper=-1.9277025234 effort=300 velocity=1
