Commit message: removing old gripper parts and adding new ones

File: ros/src/slim_description/urdf/slim_no_base.xacro (robot description, xacro)
@@ -263,7 +263,7 @@
     <material>Gazebo/Orange</material>
   </gazebo>
-  <joint name="gripper_finger_joint" type="revolute">
+  <joint name="left_finger_joint" type="revolute">
     <parent link="gripper_roll_link"/>
-    <child link="gripper_finger_link"/>
+    <child link="left_finger_link"/>
     <origin xyz="0.026 .017 0" rpy="${1.04*M_PI} ${M_PI/2} ${34.58*M_PI/180}" />
     <axis xyz="1 0 0" />
@@ -271,5 +271,44 @@
     <dynamics damping="50" friction="1"/>
   </joint>
+  <!-- new gripper -->
+  <link name="left_finger_link">
+    <inertial>
+      <origin xyz="0 0 0"  />
+      <mass value="1.0" />
+      <inertia  ixx="1.0" ixy="0.0"  ixz="0.0"  iyy="100.0"  iyz="0.0"  izz="1.0" />
+    </inertial>
+    <visual>
+      <origin xyz="0 0 0" rpy="0 0 ${M_PI}" />
+      <geometry>
+        <mesh filename="package://clam_description/stl/grippers/road_narrows/left_finger.stl" scale="${M_SCALE}" />
+      </geometry>
+      <material name="Black" />
+    </visual>
+  </link>
+  <joint name="right_finger_joint" type="revolute">
+    <parent link="gripper_roll_link"/>
+    <child link="right_finger_link"/>
+    <origin xyz="0.026 -0.011  0" rpy="${1.345*M_PI} ${M_PI/2} ${34.58*M_PI/180}" />
+    <axis xyz="1 0 0" />
+    <limit effort="300" velocity="1" lower="-3.14" upper="3.14" />
+    <mimic joint="gripper_finger_joint" multiplier="-1.0" offset="0.0" />
+    <dynamics damping="50" friction="1"/>
+  </joint>
+  <link name="right_finger_link">
+    <inertial>
+      <origin xyz="0 0 0"  />
+      <mass value="1.0" />
+      <inertia  ixx="1.0" ixy="0.0"  ixz="0.0"  iyy="100.0"  iyz="0.0"  izz="1.0" />
+    </inertial>
+    <visual>
+      <origin xyz="0 0 0" rpy="0 0 ${M_PI}" />
+      <geometry>
+        <mesh filename="package://clam_description/stl/grippers/road_narrows/right_finger.stl" scale="${M_SCALE}" />
+      </geometry>
+      <material name="Black" />
+    </visual>
+  </link>
   <!-- LEFT GRIPPER AFT LINK -->
+  <!--
   <link name="gripper_finger_link">
     <inertial>
@@ -289,14 +328,7 @@
     <material>Gazebo/Grey</material>
   </gazebo>
-  <joint name="r_gripper_aft_joint" type="fixed">
-    <parent link="gripper_roll_link"/>
-    <child link="r_gripper_aft_link"/>
-    <origin xyz="0.026 -0.011  0" rpy="${1.345*M_PI} ${M_PI/2} ${34.58*M_PI/180}" />
-    <!-- <axis xyz="1 0 0" /> -->
-    <!-- <limit effort="300" velocity="1" lower="-3.14" upper="3.14" /> -->
-    <!-- <mimic joint="gripper_finger_joint" multiplier="-1.0" offset="0.0" /> -->
-    <!-- <dynamics damping="50" friction="1"/> -->
-  </joint>
+  -->
   <!-- RIGHT GRIPPER AFT LINK -->
+  <!--
   <link name="r_gripper_aft_link">
     <inertial>
@@ -315,31 +347,4 @@
   <gazebo reference="r_gripper_aft_link">
     <material>Gazebo/Grey</material>
-  </gazebo>
-  <joint name="gripper_finger_pincher_joint" type="fixed">
-    <parent link="gripper_finger_link"/>
-    <child link="l_gripper_pincher_link"/>
-    <origin xyz="-0.0032 0 -0.0508" rpy="${203.27*M_PI/180-.3150*M_PI} 0 0" />
-    <!-- <axis xyz="1 0 0" /> -->
-    <!-- <limit effort="300" velocity="1" lower="-1.57" upper="1.57" /> -->
-    <!-- <mimic joint="gripper_finger_joint" multiplier="-1.0" offset="0.0" /> -->
-    <!-- <dynamics damping="50" friction="1"/> -->
-  </joint>
-  <!-- LEFT GRIPPER PINCHER -->
-  <link name="l_gripper_pincher_link">
-    <inertial>
-      <origin xyz="0 0 0"  />
-      <mass value="1.0" />
-      <inertia  ixx="1.0" ixy="0.0"  ixz="0.0"  iyy="100.0"  iyz="0.0"  izz="1.0" />
-    </inertial>
-    <visual>
-      <origin xyz="0 0 0" rpy="0 0 ${M_PI}" />
-      <geometry>
-        <mesh filename="package://clam_description/stl/l_gripper_pincher.STL" scale="1 1 1" />
-      </geometry>
-      <material name="Black" />
-    </visual>
-  </link>
-  <gazebo reference="l_gripper_pincher_link">
-    <material>Gazebo/Black</material>
   </gazebo>
   <joint name="r_gripper_aft_pincher_joint" type="fixed">
@@ -347,10 +352,14 @@
     <child link="r_gripper_pincher_link"/>
     <origin xyz="0 0 -0.0508" rpy="${23.27*M_PI/180-.3150*M_PI} ${M_PI} 0" />
+  -->
     <!-- <axis xyz="1 0 0" /> -->
     <!-- <limit effort="300" velocity="1" lower="0" upper="1.57" /> -->
     <!-- <mimic joint="gripper_finger_joint" multiplier="-1.0" offset="0.0" /> -->
     <!-- <dynamics damping="50" friction="1"/> -->
-  </joint>
+    <!--
+  </joint>
+    -->
   <!-- RIGHT GRIPPER PINCHER -->
+  <!--
   <link name="r_gripper_pincher_link">
     <inertial>
@@ -370,4 +379,5 @@
     <material>Gazebo/Black</material>
   </gazebo>
+  -->
   <!-- Transmissions for ROS Control -->
   <transmission name="shoulder_pan_trans">

Commit message: adding guard, low-res versions instead of redone models, model orientation

File: ros/src/slim_description/urdf/slim_no_base.xacro (robot description, xacro)
@@ -242,19 +242,20 @@
   <link name="gripper_roll_link">
     <inertial>
-      <origin xyz="0 0 0" />
-      <mass value="1.0" />
-      <inertia  ixx="1.0" ixy="0.0"  ixz="0.0"  iyy="100.0"  iyz="0.0"  izz="1.0" />
-    </inertial>
-    <visual>
-      <origin xyz="0 0 0" rpy="0 0 0" />
-      <geometry>
-        <mesh filename="package://clam_description/stl/gripper_roll_link.STL" scale="${M_SCALE}" />
-      </geometry>
-      <material name="Orange" />
-    </visual>
-    <collision>
-      <origin xyz="0 0 0" rpy="0 0 0" />
-      <geometry>
-        <mesh filename="package://clam_description/stl/gripper_roll_link.STL" scale="${M_SCALE}" />
+      <origin xyz="0.029 0.02 0.026" rpy="${M_PI} 0 0" />
+      <mass value="1.0" />
+      <inertia  ixx="1.0" ixy="0.0"  ixz="0.0"  iyy="100.0"  iyz="0.0"  izz="1.0" />
+    </inertial>
+    <visual>
+      <origin xyz="0.029 0.02 0.026" rpy="${M_PI} 0 0" />
+      <geometry>
+        <mesh filename="package://clam_description/stl/grippers/road_narrows/RNHKEF107-104-10000-faces.stl" scale="${M_SCALE}" />
+      </geometry>
+      <material name="Grey" />
+    </visual>
+    <collision>
+      <origin xyz="0.029 0.02 0.026" rpy="${M_PI} 0 0" />
+      <geometry>
+        <!-- TODO: use a cube here instead -->
+        <mesh filename="package://clam_description/stl/grippers/road_narrows/RNHKEF107-104-10000-faces.stl" scale="${M_SCALE}" />
       </geometry>
     </collision>
@@ -279,9 +280,9 @@
     </inertial>
     <visual>
-      <origin xyz="0 0 0" rpy="0 0 ${M_PI}" />
-      <geometry>
-        <mesh filename="package://clam_description/stl/grippers/road_narrows/left_finger.stl" scale="${M_SCALE}" />
-      </geometry>
-      <material name="Black" />
+      <origin xyz="-0.026 0.003 -0.002" rpy="0 ${M_PI/2} 0" />
+      <geometry>
+        <mesh filename="package://clam_description/stl/grippers/road_narrows/RNHKEF102-109-5000-faces.stl" scale="${M_SCALE}" />
+      </geometry>
+      <material name="Grey" />
     </visual>
   </link>
@@ -302,9 +303,9 @@
     </inertial>
     <visual>
-      <origin xyz="0 0 0" rpy="0 0 ${M_PI}" />
-      <geometry>
-        <mesh filename="package://clam_description/stl/grippers/road_narrows/right_finger.stl" scale="${M_SCALE}" />
-      </geometry>
-      <material name="Black" />
+      <origin xyz="-0.026 -0.031 -0.002" rpy="0 ${M_PI/2} 0" />
+      <geometry>
+        <mesh filename="package://clam_description/stl/grippers/road_narrows/RNHKEF103-109-5000-faces.stl" scale="${M_SCALE}" />
+      </geometry>
+      <material name="Grey" />
     </visual>
   </link>

Commit message: more gripper URDF updates

File: ros/src/slim_description/urdf/slim_no_base.xacro (robot description, xacro)
@@ -231,4 +231,5 @@
     <material>Gazebo/Grey</material>
   </gazebo>
+  <!-- start gripper -->
   <joint name="gripper_roll_joint" type="revolute">
     <parent link="wrist_pitch_link"/>
@@ -272,113 +273,42 @@
     <dynamics damping="50" friction="1"/>
   </joint>
-  <!-- new gripper -->
   <link name="left_finger_link">
     <inertial>
-      <origin xyz="0 0 0"  />
-      <mass value="1.0" />
-      <inertia  ixx="1.0" ixy="0.0"  ixz="0.0"  iyy="100.0"  iyz="0.0"  izz="1.0" />
-    </inertial>
-    <visual>
       <origin xyz="-0.026 0.003 -0.002" rpy="0 ${M_PI/2} 0" />
+      <mass value="1.0" />
+      <inertia  ixx="1.0" ixy="0.0"  ixz="0.0"  iyy="100.0"  iyz="0.0"  izz="1.0" />
+    </inertial>
+    <visual>
+      <origin xyz="-0.026 0.003 -0.002" rpy="0 ${M_PI/2} 0" />
       <geometry>
         <mesh filename="package://clam_description/stl/grippers/road_narrows/RNHKEF102-109-5000-faces.stl" scale="${M_SCALE}" />
       </geometry>
+      <material name="Red" />
+    </visual>
+  </link>
+  <joint name="right_finger_joint" type="revolute">
+    <parent link="gripper_roll_link" />
+    <child link="right_finger_link" />
+    <origin xyz="0.026 -0.011  0" rpy="${1.345*M_PI} ${M_PI/2} ${34.58*M_PI/180}" />
+    <axis xyz="1 0 0" />
+    <mimic joint="left_finger_joint" multiplier="-1.0" offset="0.0" />
+    <limit effort="300" velocity="1" lower="-1.8254371376" upper="0.0"/>
+    <dynamics damping="50" friction="1"/>
+  </joint>
+  <link name="right_finger_link">
+    <inertial>
+      <origin xyz="0 0 0" />
+      <mass value="1.0" />
+      <inertia  ixx="1.0" ixy="0.0"  ixz="0.0"  iyy="100.0"  iyz="0.0"  izz="1.0" />
+    </inertial>
+    <visual>
+      <origin xyz="-0.026 -0.031 -0.002" rpy="0 ${M_PI/2} 0" />
+      <geometry>
+        <mesh filename="package://clam_description/stl/grippers/road_narrows/RNHKEF103-109-5000-faces.stl" scale="${M_SCALE}" />
+      </geometry>
       <material name="Grey" />
     </visual>
   </link>
-  <joint name="right_finger_joint" type="revolute">
-    <parent link="gripper_roll_link"/>
-    <child link="right_finger_link"/>
-    <origin xyz="0.026 -0.011  0" rpy="${1.345*M_PI} ${M_PI/2} ${34.58*M_PI/180}" />
-    <axis xyz="1 0 0" />
-    <limit effort="300" velocity="1" lower="-3.14" upper="3.14" />
-    <mimic joint="gripper_finger_joint" multiplier="-1.0" offset="0.0" />
-    <dynamics damping="50" friction="1"/>
-  </joint>
-  <link name="right_finger_link">
-    <inertial>
-      <origin xyz="0 0 0"  />
-      <mass value="1.0" />
-      <inertia  ixx="1.0" ixy="0.0"  ixz="0.0"  iyy="100.0"  iyz="0.0"  izz="1.0" />
-    </inertial>
-    <visual>
-      <origin xyz="-0.026 -0.031 -0.002" rpy="0 ${M_PI/2} 0" />
-      <geometry>
-        <mesh filename="package://clam_description/stl/grippers/road_narrows/RNHKEF103-109-5000-faces.stl" scale="${M_SCALE}" />
-      </geometry>
-      <material name="Grey" />
-    </visual>
-  </link>
-  <!-- LEFT GRIPPER AFT LINK -->
-  <!--
-  <link name="gripper_finger_link">
-    <inertial>
-      <origin xyz="0 0 0"  />
-      <mass value="1.0" />
-      <inertia  ixx="1.0" ixy="0.0"  ixz="0.0"  iyy="100.0"  iyz="0.0"  izz="1.0" />
-    </inertial>
-    <visual>
-      <origin xyz="0 0 0" rpy="0 0 ${M_PI}" />
-      <geometry>
-        <mesh filename="package://clam_description/stl/l_gripper_aft_link.STL" scale="1 1 1" />
-      </geometry>
-      <material name="Grey" />
-    </visual>
-  </link>
-  <gazebo reference="l_gripper_aft_link">
-    <material>Gazebo/Grey</material>
-  </gazebo>
-  -->
-  <!-- RIGHT GRIPPER AFT LINK -->
-  <!--
-  <link name="r_gripper_aft_link">
-    <inertial>
-      <origin xyz="0 0 0"  />
-      <mass value="1.0" />
-      <inertia  ixx="1.0" ixy="0.0"  ixz="0.0"  iyy="100.0"  iyz="0.0"  izz="1.0" />
-    </inertial>
-    <visual>
-      <origin xyz="0 0 0" rpy="0 0 ${M_PI}" />
-      <geometry>
-        <mesh filename="package://clam_description/stl/r_gripper_aft_link.STL" scale="1 1 1" />
-      </geometry>
-      <material name="Grey" />
-    </visual>
-  </link>
-  <gazebo reference="r_gripper_aft_link">
-    <material>Gazebo/Grey</material>
-  </gazebo>
-  <joint name="r_gripper_aft_pincher_joint" type="fixed">
-    <parent link="r_gripper_aft_link"/>
-    <child link="r_gripper_pincher_link"/>
-    <origin xyz="0 0 -0.0508" rpy="${23.27*M_PI/180-.3150*M_PI} ${M_PI} 0" />
-  -->
-    <!-- <axis xyz="1 0 0" /> -->
-    <!-- <limit effort="300" velocity="1" lower="0" upper="1.57" /> -->
-    <!-- <mimic joint="gripper_finger_joint" multiplier="-1.0" offset="0.0" /> -->
-    <!-- <dynamics damping="50" friction="1"/> -->
-    <!--
-  </joint>
-    -->
-  <!-- RIGHT GRIPPER PINCHER -->
-  <!--
-  <link name="r_gripper_pincher_link">
-    <inertial>
-      <origin xyz="0 0 0" />
-      <mass value="1.0" />
-      <inertia  ixx="1.0" ixy="0.0"  ixz="0.0"  iyy="100.0"  iyz="0.0"  izz="1.0" />
-    </inertial>
-    <visual>
-      <origin xyz="0 0 0" rpy="0 0 ${M_PI}" />
-      <geometry>
-        <mesh filename="package://clam_description/stl/r_gripper_pincher.STL" scale="1 1 1" />
-      </geometry>
-      <material name="Black" />
-    </visual>
-  </link>
-  <gazebo reference="r_gripper_pincher_link">
-    <material>Gazebo/Black</material>
-  </gazebo>
-  -->
+  <!-- end gripper -->
   <!-- Transmissions for ROS Control -->
   <transmission name="shoulder_pan_trans">
@@ -454,5 +384,5 @@
   <transmission name="gripper_finger_trans">
     <type>transmission_interface/SimpleTransmission</type>
-    <joint name="gripper_finger_joint">
+    <joint name="left_finger_joint">
       <hardwareInterface>PositionJointInterface</hardwareInterface>
     </joint>

Commit message: aligning joints in URDF

File: ros/src/slim_description/urdf/slim_no_base.xacro (robot description, xacro)
@@ -268,5 +268,5 @@
     <parent link="gripper_roll_link"/>
     <child link="left_finger_link"/>
-    <origin xyz="0.026 .017 0" rpy="${1.04*M_PI} ${M_PI/2} ${34.58*M_PI/180}" />
+    <origin xyz="0.041 .02 0" rpy="4.1 ${M_PI/2} ${34.58*M_PI/180}" />
     <axis xyz="1 0 0" />
     <limit effort="300" velocity="1" lower="-1.8254371376" upper="0.0"/>
@@ -280,9 +280,9 @@
     </inertial>
     <visual>
-      <origin xyz="-0.026 0.003 -0.002" rpy="0 ${M_PI/2} 0" />
+      <origin xyz="-0.026 -0.00 0.012" rpy="0 ${M_PI/2} 0" />
       <geometry>
         <mesh filename="package://clam_description/stl/grippers/road_narrows/RNHKEF102-109-5000-faces.stl" scale="${M_SCALE}" />
       </geometry>
-      <material name="Red" />
+      <material name="Grey" />
     </visual>
   </link>
@@ -290,5 +290,5 @@
     <parent link="gripper_roll_link" />
     <child link="right_finger_link" />
-    <origin xyz="0.026 -0.011  0" rpy="${1.345*M_PI} ${M_PI/2} ${34.58*M_PI/180}" />
+    <origin xyz="0.04 -0.021 0" rpy="4 ${M_PI/2} ${34.58*M_PI/180}" />
     <axis xyz="1 0 0" />
     <mimic joint="left_finger_joint" multiplier="-1.0" offset="0.0" />
@@ -303,9 +303,9 @@
     </inertial>
     <visual>
-      <origin xyz="-0.026 -0.031 -0.002" rpy="0 ${M_PI/2} 0" />
+      <origin xyz="-0.026 -0.041 0.012" rpy="0 ${M_PI/2} 0" />
       <geometry>
         <mesh filename="package://clam_description/stl/grippers/road_narrows/RNHKEF103-109-5000-faces.stl" scale="${M_SCALE}" />
       </geometry>
-      <material name="Grey" />
+      <material name="Red" />
     </visual>
   </link>
